File: Card_CRAN_SEGULA/Connections_3_sch.kicad_sch (KiCad schematic)
At the start: 14 parts, among them J11 530480410, J12 530480410, J13 530480410, J14 530480410, J15 530480410, J16 530480610, J8 530480910, J9 530480410

Commit message: Carte presque fini avant la dernière vérification
Parts:
- removed J8: 530480910, pin_9x1_0530480910:CONN09_530480910_MOL, symbol pin_9x1_0530480910:530480910
- removed R47: 10kR, Resistor_10kR_CRGP0402F10K:RESC1105X40N, symbol Resistor:R
- removed R48, R49: 0R, Resistor_0R_RCS06030000Z0EC:RESC1508X50N, symbol Resistor:R
- added H1, H2, H3, H4: MountingHole_Pad, Mounting_Hole_M3:MountingHole_3.2mm_M3_Pad_Via, symbol mountinghole_pad:MountingHole_Pad
Connections:
- net +3.3V is gone; now on net +3V3: J12.1, J14.1, J16.1, J9.1, R61.1
- net +3V3: now also J15.1
- net GND: now also H1.1, H2.1, H3.1, H4.1
Other:
- note added: "Connectors (Additional peripherals + Mounting + (NAV <-> COM))"
- note added: "Mounting Hole"
- note added: "SPI (NAV <-> COM)"
- note added: "UART (NAV <-> COM)"
- note removed: "Connections (NAV <-> COM)"
- note removed: "Connectors (Additional peripherals)"
- note removed: "I2C Connections"
- note removed: "SPI Connections"
- note removed: "UART Connections"
- moved on the sheet: J14, J9
