File: Card_CRAN_SEGULA/MCU_Communication.kicad_sch (KiCad schematic)
At the start: 37 parts, among them IC2 STM32H753VIT6, SW4 TDD01H0SB1R, SW5 SMD-BUTTON_4P-5.2X5.2X1.5MM-S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, X2 ABM8G-25.000MHZ-4Y-T3

Commit message: Carte presque fini avant la dernière vérification
Parts:
- removed R58, R59: 4.7kR, Resistor_4_7kR_SG73P1ETTP4701F:RESC1005X40N, symbol Resistor:R
Connections:
- net +3.3V is gone; now on net +3V3: C54.1, C55.1, C56.1, C57.1, C58.1, C59.1, C60.1, C61.1, C62.1, C63.1, C64.1, C65.1, FB10.2, IC2.100 (VDD), IC2.11 (VDD), IC2.27 (VDD), IC2.50 (VDD), IC2.6 (VBAT), IC2.75 (VDD), R53.1, R54.1, R55.1, R56.1
- net WIFI_INT: now reaches IC2.33 (PC5)
- net WIFI_BUCKEN: now reaches IC2.63 (PC6)
- net GPIO_A_COM: no longer names the net of IC2.81 (PD0)
- net GPIO_B_COM: no longer names the net of IC2.82 (PD1)
- net GPIO_C_COM: no longer names the net of IC2.83 (PD2)
- net GPIO_D_COM: no longer names the net of IC2.84 (PD3)
- net GPIO_E_COM: no longer names the net of IC2.85 (PD4)
- net GPIO_F_COM: no longer names the net of IC2.86 (PD5)
- net GPIO_G_COM: no longer names the net of IC2.87 (PD6)
- net GPIO_H_COM: no longer names the net of IC2.88 (PD7)
- net I2C3_SDA_COM: no longer names the net of IC2.66 (PC9)
- net I2C3_SLC_COM: no longer names the net of IC2.67 (PA8)
- net LED_A_COM: no longer names the net of IC2.34 (PB0)
- net LED_B_COM: no longer names the net of IC2.35 (PB1)
- net LED_C_COM: no longer names the net of IC2.36 (PB2)
- no-connect marks 0 -> 39
Other:
- moved on the sheet: R53, R54, R55, R56
