File: Card_CRAN_SEGULA/MCU_Navigation.kicad_sch (KiCad schematic)
At the start: 38 parts, among them IC1 STM32F405RGT6, SW1 TDD01H0SB1R, SW2 TDD01H0SB1R, SW3 SMD-BUTTON_4P-5.2X5.2X1.5MM-S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, X3 ABM8G-25.000MHZ-4Y-T3

Commit message: Carte presque fini avant la dernière vérification
Connections:
- net +3.3V is gone; now on net +3V3: C37.1, C38.1, C39.1, C40.1, C41.1, C42.1, C43.1, C44.1, C45.1, C46.1, FB9.1, R36.1, R37.1, R38.1, R39.1, SW1.1, SW2.1
- net LED_C_NAV: now also D14.2 (A)
- net GPIO_D_NAV: no longer names the net of IC1.30 (PB11)
- net I2C3_SDA_NAV: no longer names the net of IC1.40 (PC9)
- net I2C3_SLC_NAV: no longer names the net of IC1.41 (PA8)
- no-connect marks 5 -> 12
Other:
- note removed: "I2C3_NAV already pulled up by I2C3_COM resistors"
