File: Card_CRAN_SEGULA/Card_CRAN_SEGULA.kicad_pcb (KiCad board)
At the start: 4 copper layers, 150 x 70 mm, 241 parts, among them IC1 STM32F405RGT6, IC2 STM32H753VIT6, J1 503398-1892, J11 530480410, J12 530480410, J13 530480410, J14 530480410, J15 530480410, J16 530480610, J2 USB4110GFA, J3 USB4110GFA, J4 USB4110GFA, J5 USB4110GFA, J6 M50-3600542R, J7 M50-3600542R, J8 530480910, J9 530480410, SW1 TDD01H0SB1R, SW2 TDD01H0SB1R, SW3 SMD-BUTTON_4P-5.2X5.2X1.5MM-S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, SW4 TDD01H0SB1R, SW5 SMD-BUTTON_4P-5.2X5.2X1.5MM-S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, U1 IIS2MDCTR, U10 CP2102N-A02-GQFN20R, U11 INA219AIDCNR, U12 LD39200PU33R, U2 IIM-42652, U3 NEO-M9N-00B, U4 24CW1280T-I/OT, U5 24CW1280T-I/OT, U6 NRF7002-QFAA-R, U7 W25N01GVZEIG_TR, U8 DPX165950DT-8148A1, U9 CP2102N-A02-GQFN20R, X1 NX2016SA-40M-STD-CZS-3, X2 ABM8G-25.000MHZ-4Y-T3, X3 ABM8G-25.000MHZ-4Y-T3

Commit message: Carte presque fini avant la dernière vérification
Parts:
- removed J8: 530480910, pin_9x1_0530480910:CONN09_530480910_MOL
- removed R47: 10kR, Resistor_10kR_CRGP0402F10K:RESC1105X40N
- removed R48, R49: 0R, Resistor_0R_RCS06030000Z0EC:RESC1508X50N
- removed R58, R59: 4.7kR, Resistor_4_7kR_SG73P1ETTP4701F:RESC1005X40N
- added C13: 0.47uF, Capacitor_0_47uF_GRM033R60J474KE90D:CAPC0603X33N, F.Cu at (58.6, 138.6)
- added C14: 4.7uF, Capacitor_4_7uF_GRM188C81E475KE11D:CAPC1608X100N, F.Cu at (57.1, 140.1)
- added C17: 22nF, Capacitor_22nF_10V_GRM033R61A223KE84D:CAPC0603X33N, F.Cu at (63.4, 139.1)
- added C23: 0.47uF, Capacitor_0_47uF_GRM033R60J474KE90D:CAPC0603X33N, F.Cu at (79.7, 132.0)
- added C24: 4.7uF, Capacitor_4_7uF_GRM188C81E475KE11D:CAPC1608X100N, F.Cu at (79.6, 134.0)
- added C25: 4.7uF, Capacitor_4_7uF_GRM188C81E475KE11D:CAPC1608X100N, F.Cu at (75.7, 136.7)
- added C27: 4.7uF, Capacitor_4_7uF_GRM188C81E475KE11D:CAPC1608X100N, F.Cu at (62.0, 139.8)
- added C28: 0.22uF, Capacitor_0_22uF_GRM033R61A224KE90D:CAPC0603X33N, F.Cu at (64.4, 140.8)
- added H1: MountingHole_Pad, Mounting_Hole_M3:MountingHole_3.2mm_M3_Pad_Via, F.Cu at (55.0, 85.0)
- added H2: MountingHole_Pad, Mounting_Hole_M3:MountingHole_3.2mm_M3_Pad_Via, F.Cu at (185.0, 85.0)
- added H3: MountingHole_Pad, Mounting_Hole_M3:MountingHole_3.2mm_M3_Pad_Via, F.Cu at (55.0, 145.0)
- added H4: MountingHole_Pad, Mounting_Hole_M3:MountingHole_3.2mm_M3_Pad_Via, F.Cu at (185.0, 145.0)
- added L2: 3.3uH, Inductor_3_3uH_74479775233:WE-PMI_0805_H1, F.Cu at (76.1, 134.9)
- C12, C35, C47, C48, C53, C71, C72, D12, D13, D14, FB9, R3, R36, R37, R38, R39, R46, R50, R51, R61, R65: moved to B.Cu
- C15: footprint Capacitor_100nF_GRM155C71H104JE19D:CAPC1005X55N -> Capacitor_100nF_16V_GRM033C71C104KE14D:CAPC0603X33N; moved to F.Cu
- C16: footprint Capacitor_2.2uF_GRM188R61H225KE11D:CAPC1608X100N -> Capacitor_2_2uF_16V_GRM188C71C225KE11J:CAPC1608X100N; moved to F.Cu
- C18: footprint Capacitor_1uF_C0603C105Z3VACTU:CAPC17595_90N_KEM -> Capacitor_1uF_10V_GCM155C71A105KE38D:CAPC1005X70N; moved to F.Cu
- C20: footprint Capacitor_100nF_GRM155C71H104JE19D:CAPC1005X55N -> Capacitor_100nF_16V_GRM033C71C104KE14D:CAPC0603X33N
- C21: footprint Capacitor_2.2uF_GRM188R61H225KE11D:CAPC1608X100N -> Capacitor_2_2uF_25V_GRM155R61E225KE11D:CAPC1005X70N
- C22: footprint Capacitor_1uF_C0603C105Z3VACTU:CAPC17595_90N_KEM -> Capacitor_1uF_16V_GRM155C81C105KE11D:CAPC1005X60N; moved to F.Cu
- C26: footprint Capacitor_1uF_C0603C105Z3VACTU:CAPC17595_90N_KEM -> Capacitor_1uF_GRM155R6YA105KE11D:CAPC1005X60N
- C29, C30: footprint Capacitor_2.2uF_GRM188R61H225KE11D:CAPC1608X100N -> Capacitor_2_2uF_16V_GRM188C71C225KE11J:CAPC1608X100N
- C31, C32, C52, C69, C70, D4, D8, FB10, FB4, FB8, J1, R10, R12: moved to F.Cu
- J2, J3, J4, J5: footprint USB_C_USB4110GFA:GCT_USB4110GFA -> USB_C_USB4110GFA:USB4110-GF-A_GCT; moved to F.Cu
- REG1: footprint MIC26903YJL-TR:MLF28_5X6_MCH -> MIC26903YJL-TR:MIC24054YJLTR
- U1: footprint IIS2MDCTR:LGA-12_2X2X0P7_STM -> IIS2MDCTR:IIS2MDCTR
- U10: footprint UART_TO_USB_CP2102N-A02-GQFN20R:SILABS_CP2102N-A02-GQFN20R -> UART_TO_USB_CP2102N-A02-GQFN20R:QFN20_SIL
- U9: footprint UART_TO_USB_CP2102N-A02-GQFN20R:SILABS_CP2102N-A02-GQFN20R -> UART_TO_USB_CP2102N-A02-GQFN20R:QFN20_SIL; moved to F.Cu
- moved JP1 403.3 mm to (187.5, 91.4), turned to 180 degrees
- moved D9 386.4 mm to (140.2, 90.8)
- moved D8 386.0 mm to (152.0, 91.2)
- moved FB7 385.1 mm to (139.5, 92.6)
- moved FB8 384.6 mm to (152.4, 93.2), turned to 0 degrees
- moved D4 381.8 mm to (166.8, 92.8), turned to 180 degrees
- moved D5 380.7 mm to (155.6, 92.8), turned to 0 degrees
- moved JP5 378.5 mm to (166.8, 90.4)
- moved U10 377.1 mm to (147.2, 97.8), turned to -90 degrees
- moved C34 375.8 mm to (135.4, 99.0), turned to 180 degrees
- moved JP6 375.0 mm to (183.4, 112.8)
- moved JP4 373.6 mm to (155.6, 90.4), turned to 180 degrees
- moved FB3 373.5 mm to (155.6, 94.8), turned to 90 degrees
- moved FB4 373.4 mm to (166.8, 94.8), turned to -90 degrees
- moved C39 362.8 mm to (139.0, 114.0), turned to 180 degrees
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Connections:
- C3 pad 1: +3V3 -> WIFI_BUCVBATS
- C4 pad 1: +3V3 -> WIFI_BUCVBATS
- C73 pad 2: +3V3 -> WIFI_BUCVBATS
- C8 pad 2: +3V3 -> WIFI_BUCVBATS
- D14 pad 2: unconnected-(D14-A-Pad2) -> LED_C_NAV
- IC1 pad 1: +3V3 -> WIFI_BUCVBATS
- IC1 pad 19: +3V3 -> WIFI_BUCVBATS
- IC1 pad 30: GPIO_D_NAV -> unconnected-(IC1-PB11-Pad30)
- IC1 pad 32: +3V3 -> WIFI_BUCVBATS
- IC1 pad 40: I2C3_SDA_NAV -> unconnected-(IC1-PC9-Pad40)
- IC1 pad 41: I2C3_SLC_NAV -> unconnected-(IC1-PA8-Pad41)
- IC1 pad 48: +3V3 -> WIFI_BUCVBATS
- IC1 pad 64: +3V3 -> WIFI_BUCVBATS
- IC2 pad 33: unconnected-(IC2-PC5-Pad33) -> WIFI_INT
- IC2 pad 34: LED_A_COM -> unconnected-(IC2-PB0-Pad34)
- IC2 pad 35: LED_B_COM -> unconnected-(IC2-PB1-Pad35)
- IC2 pad 36: LED_C_COM -> unconnected-(IC2-PB2-Pad36)
- IC2 pad 63: unconnected-(IC2-PC6-Pad63) -> WIFI_BUCKEN
- IC2 pad 66: I2C3_SDA_COM -> unconnected-(IC2-PC9-Pad66)
- IC2 pad 67: I2C3_SLC_COM -> unconnected-(IC2-PA8-Pad67)
- IC2 pad 81: GPIO_A_COM -> unconnected-(IC2-PD0-Pad81)
- IC2 pad 82: GPIO_B_COM -> unconnected-(IC2-PD1-Pad82)
- IC2 pad 83: GPIO_C_COM -> unconnected-(IC2-PD2-Pad83)
- IC2 pad 84: GPIO_D_COM -> unconnected-(IC2-PD3-Pad84)
- IC2 pad 85: GPIO_E_COM -> unconnected-(IC2-PD4-Pad85)
- IC2 pad 86: GPIO_F_COM -> unconnected-(IC2-PD5-Pad86)
- IC2 pad 87: GPIO_G_COM -> unconnected-(IC2-PD6-Pad87)
- IC2 pad 88: GPIO_H_COM -> unconnected-(IC2-PD7-Pad88)
- J1 pad 10: SD_SWITCH -> unconnected-(J1-DETECT_SWITCH-Pad10)
- J11 pad 1: +3V3 -> WIFI_BUCVBATS
- J13 pad 1: +3V3 -> WIFI_BUCVBATS
- J15 pad 1: unconnected-(J15-Pad1) -> WIFI_BUCVBATS
- J2 pad A4/B9: Net-(D5-A) -> Net-(D4-A)
- J3 pad A4/B9: Net-(D3-A) -> Net-(D2-A)
- JP1 pad 1: +3V3 -> WIFI_BUCVBATS
- R12 pad 1: USB_DP_COM -> USB_DN_COM
- R12 pad 2: Net-(J3-DP2) -> Net-(J3-DN2)
- R13 pad 1: Net-(J3-DN2) -> Net-(J3-DP2)
- R13 pad 2: USB_DN_COM -> USB_DP_COM
- R15 pad 1: Net-(J2-DN2) -> Net-(J2-DP2)
- R15 pad 2: USB_DN_NAV -> USB_DP_NAV
- R16 pad 1: USB_DP_NAV -> USB_DN_NAV
- R16 pad 2: Net-(J2-DP2) -> Net-(J2-DN2)
- R2 pad 1: +3V3 -> WIFI_BUCVBATS
- R3 pad 1: +3V3 -> WIFI_BUCVBATS
- R4 pad 1: +3V3 -> WIFI_BUCVBATS
- R42 pad 1: +3V3 -> WIFI_BUCVBATS
- SW4 pad 1: +3V3 -> WIFI_BUCVBATS
- U1 pad 3: +3V3 -> WIFI_BUCVBATS
- U1 pad 9: +3V3 -> WIFI_BUCVBATS
- U11 pad 4: +3V3 -> WIFI_BUCVBATS
- U3 pad 23: +3V3 -> WIFI_BUCVBATS
Routing:
- net +5V: track 0.00 -> 651.8 mm, vias 0 -> 16
- net GND: track 0.00 -> 341.2 mm, vias 0 -> 311
- net WIFI_BUCVBATS: track 0.00 -> 327.6 mm, vias 0 -> 49
- net NRST_COM: track 0.00 -> 74.7 mm, vias 0 -> 2
- net UART1_RX_COM: track 0.00 -> 65.8 mm, vias 0 -> 2
- net UART1_TX_COM: track 0.00 -> 61.7 mm, vias 0 -> 2
- net NRST_NAV: track 0.00 -> 60.2 mm, vias 0 -> 2
- net GNSS_NRST: track 0.00 -> 58.7 mm, vias 0 -> 2
- net REG_VIN: track 0.00 -> 58.6 mm, vias 0 -> 2
- net GNSS_PPS: track 0.00 -> 57.8 mm, vias 0 -> 4
- net I2C_SCL_NAV: track 0.00 -> 53.3 mm, vias 0 -> 3
- net WIFI_BUCKEN: track 0.00 -> 52.8 mm, vias 0 -> 2
- net I2C_SDA_NAV: track 0.00 -> 50.9 mm, vias 0 -> 3
- net WIFI_INT: track 0.00 -> 49.7 mm, vias 0 -> 2
- net USB_VBUS_NAV: track 0.00 -> 49.5 mm, vias 0 -> 3
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- added copper zone on F.Cu, net +5V
- added copper zone on B.Cu, net GND
- added copper zone on F.Cu, net GND
- added copper zone on F.Cu, net REG_CS
- added copper zone on B.Cu, net REG_FB
- added copper zone on F.Cu, net REG_FB
- added copper zone on F.Cu, net REG_VIN
- added copper zone on F.Cu, net VIN+
- added copper zone on In2.Cu, net WIFI_BUCVBATS
- removed copper zone on In2.Cu, net +3V3
Other:
- board size 150 x 70 mm -> 140 x 70 mm
- rule pad_to_mask_clearance: 0.08 -> 0

Commit message: MàJ 07/07/2025
Parts:
- removed D2, D4, D6, D8: SD103AWS, D_Schottky_SD103AWS:D_SOD-323
- removed FB2, FB4, FB6, FB8: FerriteBead_Small, FERRITE_BEAD_120_OHM_0402_4LN_MPZ1005S121HT000:L_0402_1005Metric
- removed JP3, JP5: SolderJumper_2_Open, SolderJumper_2_Open:SolderJumper-2_P1.3mm_Open_RoundedPad1.0x1.5mm
- removed R10, R11, R12, R13, R15, R16, R6, R7: 22R, Resistor_22R_ERA-2AKD220X:RES_ERA2AKD220X
- added U13: USBLC6-2SC6, Package_TO_SOT_SMD:SOT-23-6, F.Cu at (161.2, 95.3)
- added U14: USBLC6-2SC6, Package_TO_SOT_SMD:SOT-23-6, F.Cu at (127.0, 134.0)
- C31, C32: moved to B.Cu
- R2: value 10R -> 10kR; footprint Resistor_10R_ERA-2AKD100X:RES_ERA2AKD100X -> Resistor_10kR_CRGP0402F10K:RESC1105X40N
- moved JP2 13.1 mm to (120.5, 138.6), turned to 180 degrees
- moved D3 11.5 mm to (121.6, 136.0)
- moved FB1 11.3 mm to (120.4, 134.4)
- moved R2 1.70 mm to (179.4, 90.3), turned to -90 degrees
- moved JP4 0.95 mm to (154.6, 90.4)
- moved U8 0.74 mm to (56.1, 133.7)
- moved C32 0.57 mm to (116.2, 126.6)
- moved C88 0.07 mm to (119.0, 132.1)
Connections:
- J2 pad A4/B9: Net-(D4-A) -> Net-(D5-A)
- J2 pad B6: Net-(J2-DP2) -> Net-(J2-DP1)
- J2 pad B7: Net-(J2-DN2) -> Net-(J2-DN1)
- J3 pad A4/B9: Net-(D2-A) -> Net-(D3-A)
- J3 pad B6: Net-(J3-DP2) -> Net-(J3-DP1)
- J3 pad B7: Net-(J3-DN2) -> Net-(J3-DN1)
Routing:
- net +5V: track 651.8 -> 486.2 mm
- net USB_VBUS_NAV: track 49.5 -> 27.1 mm, vias 3 -> 2
- net USB_VBUS_COM: track 44.7 -> 27.1 mm, vias 3 -> 2
- net Net-(D3-A): track 8.60 -> 25.3 mm, vias 0 -> 2
- net Net-(D5-A): track 7.37 -> 21.8 mm, vias 0 -> 2
- net USB_DN_COM: track 31.3 -> 22.2 mm, vias 3 -> 0
- net USB_DN_NAV: track 35.2 -> 27.2 mm, vias 2 -> 0
- net GND: track 341.2 -> 348.9 mm, vias 311 -> 336
- net Net-(D2-A): track 7.58 -> 0.00 mm
- net Net-(D4-A): track 7.53 -> 0.00 mm
- net USB_DP_COM: track 31.3 -> 24.6 mm, vias 2 -> 0
- net UART_DP_COM: track 21.9 -> 15.3 mm, vias 3 -> 0
- net Net-(J2-DN2): track 6.52 -> 0.00 mm
- net Net-(J3-DN2): track 6.51 -> 0.00 mm
- net Net-(J3-DP2): track 6.51 -> 0.00 mm
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