File: Card_CRAN_SEGULA/Communication_Peripherique.kicad_sch (KiCad schematic)
At the start: 33 parts, among them U5 24CW1280T-I/OT, U6 NRF7002-QFAA-R, U7 W25N01GVZEIG_TR, U8 DPX165950DT-8148A1, X1 NX2016SA-40M-STD-CZS-3

Commit message: Carte presque fini avant la dernière vérification
Parts:
- C13, C23: footprint (none) -> Capacitor_0_47uF_GRM033R60J474KE90D:CAPC0603X33N
- C14, C24, C25, C27: footprint (none) -> Capacitor_4_7uF_GRM188C81E475KE11D:CAPC1608X100N
- C15, C20: footprint Capacitor_100nF_GRM155C71H104JE19D:CAPC1005X55N -> Capacitor_100nF_16V_GRM033C71C104KE14D:CAPC0603X33N
- C16, C29, C30: footprint Capacitor_2.2uF_GRM188R61H225KE11D:CAPC1608X100N -> Capacitor_2_2uF_16V_GRM188C71C225KE11J:CAPC1608X100N
- C17: footprint (none) -> Capacitor_22nF_10V_GRM033R61A223KE84D:CAPC0603X33N
- C18: footprint Capacitor_1uF_C0603C105Z3VACTU:CAPC17595_90N_KEM -> Capacitor_1uF_10V_GCM155C71A105KE38D:CAPC1005X70N
- C21: footprint Capacitor_2.2uF_GRM188R61H225KE11D:CAPC1608X100N -> Capacitor_2_2uF_25V_GRM155R61E225KE11D:CAPC1005X70N
- C22: footprint Capacitor_1uF_C0603C105Z3VACTU:CAPC17595_90N_KEM -> Capacitor_1uF_16V_GRM155C81C105KE11D:CAPC1005X60N
- C26: footprint Capacitor_1uF_C0603C105Z3VACTU:CAPC17595_90N_KEM -> Capacitor_1uF_GRM155R6YA105KE11D:CAPC1005X60N
- C28: footprint (none) -> Capacitor_0_22uF_GRM033R61A224KE90D:CAPC0603X33N
- L2: footprint (none) -> Inductor_3_3uH_74479775233:WE-PMI_0805_H1
Connections:
- net +3.3V is gone; now on net +3V3: C11.1, C12.2, C25.1, C26.2, C27.2, C29.1, C30.2, R43.1, U5.4 (VCC), U6.13 (VBAT), U6.20 (AFEVBAT), U6.25 (BUCKVBAT), U6.31 (BUCVBATS), U6.48 (IOVDD), U7.8 (VCC)
