File: Card_CRAN_SEGULA/Connections.kicad_sch (KiCad schematic)
At the start: 34 parts, among them J1 503398-1892, J2 USB4110GFA, J3 USB4110GFA, J6 M50-3600542R, J7 M50-3600542R

Commit message: Carte presque fini avant la dernière vérification
Parts:
- J2, J3: footprint USB_C_USB4110GFA:GCT_USB4110GFA -> USB4110-GF-A_GCT; symbol USB_C_USB4110GFA:USB4110GFA -> USB4110GFA:USB4110-GF-A
Connections:
- net GND: now also J2.15 (S1), J2.16 (S2), J2.17 (S3), J2.18 (S4), J2.A12/B1 (GND), J3.15 (S1), J3.16 (S2), J3.17 (S3), J3.18 (S4), J3.A12/B1 (GND); no longer J2.B1/A12 (GND__1), J2.S1 (GND__2), J2.S2 (GND__3), J2.S3 (GND__4), J2.S4 (GND__5), J3.B1/A12 (GND__1), J3.S1 (GND__2), J3.S2 (GND__3), J3.S3 (GND__4), J3.S4 (GND__5)
- net USB_DN_COM: now also R12.1; no longer R13.2
- net USB_DN_NAV: now also R16.1; no longer R15.2
- net USB_DP_COM: now also R13.2; no longer R12.1
- net USB_DP_NAV: now also R15.2; no longer R16.1
- net at D3.2 (A), JP2.1 (A): now also J3.A9/B4 (VBUS); no longer J3.A4/B9 (VBUS)
- net at R16.2: now also J2.B7 (DN2); no longer J2.B6 (DP2)
- net at R12.2: now also J3.B7 (DN2); no longer J3.B6 (DP2)
- net at D5.2 (A), JP4.1 (A): now also J2.A9/B4 (VBUS); no longer J2.A4/B9 (VBUS)
- net at D2.2 (A), JP3.1 (A): now also J3.A4/B9 (VBUS); no longer J3.B4/A9 (VBUS__1)
- net at D4.2 (A), JP5.1 (A): now also J2.A4/B9 (VBUS); no longer J2.B4/A9 (VBUS__1)
- net at R13.1: now also J3.B6 (DP2); no longer J3.B7 (DN2)
- net at R15.1: now also J2.B6 (DP2); no longer J2.B7 (DN2)
- net +3.3V renamed +3V3
- net SD_SWITCH: no longer names the net of J1.10 (DETECT_SWITCH)
- no-connect marks 8 -> 9
Other:
- moved on the sheet: R10, R11, R23, R24, R25, R6, R7, R8, R9

Commit message: MàJ 07/07/2025
Parts:
- removed D2, D4: SD103AWS, D_Schottky_SD103AWS:D_SOD-323, symbol schottky_SD103AWS:D_Schottky
- removed FB2, FB4: FerriteBead_Small, FERRITE_BEAD_120_OHM_0402_4LN_MPZ1005S121HT000:L_0402_1005Metric, symbol ferritebead_small:FerriteBead_Small
- removed JP3, JP5: SolderJumper_2_Open, SolderJumper_2_Open:SolderJumper-2_P1.3mm_Open_RoundedPad1.0x1.5mm, symbol solderjumper_2_open:SolderJumper_2_Open
- removed R10, R11, R12, R13, R15, R16, R6, R7: 22R, Resistor_22R_ERA-2AKD220X:RES_ERA2AKD220X, symbol Resistor:R
- added U13, U14: USBLC6-2SC6, Package_TO_SOT_SMD:SOT-23-6, symbol Power_Protection:USBLC6-2SC6
Connections:
- net +5V: now also U13.5 (VBUS), U14.5 (VBUS)
- net GND: now also U13.2 (GND), U14.2 (GND)
- net USB_DN_COM: now also U14.6 (I/O1)
- net USB_DN_NAV: now also U13.6 (I/O1)
- net USB_DP_COM: now also U14.4 (I/O2)
- net USB_DP_NAV: now also U13.4 (I/O2)
- net at D3.2 (A), J3.A9/B4 (VBUS), JP2.1 (A): now also J3.A4/B9 (VBUS)
- net at J2.B7 (DN2): now also J2.A7 (DN1), U13.1 (I/O1)
- net at J3.B7 (DN2): now also J3.A7 (DN1), U14.1 (I/O1)
- net at D5.2 (A), J2.A9/B4 (VBUS), JP4.1 (A): now also J2.A4/B9 (VBUS)
- net at J3.A6 (DP1): now also J3.B6 (DP2), U14.3 (I/O2)
- net at J2.A6 (DP1): now also J2.B6 (DP2), U13.3 (I/O2)
Other:
- moved on the sheet: D3, FB1, R17, R22
