File: Card_CRAN_SEGULA/Navigation_Peripherique.kicad_sch (KiCad schematic)
At the start: 22 parts, among them U1 IIS2MDCTR, U2 IIM-42652, U3 NEO-M9N-00B, U4 24CW1280T-I/OT

Commit message: Carte presque fini avant la dernière vérification
Parts:
- U1: footprint IIS2MDCTR:LGA-12_2X2X0P7_STM -> IIS2MDCTR:IIS2MDCTR
Connections:
- net +3.3V is gone; now on net +3V3: C10.1, C2.1, C5.1, C6.1, C7.1, R44.1, R45.2, U1.10 (VDD_IO), U2.5 (VDDIO), U2.8 (VDD), U4.4 (VCC)
Other:
- note added: "GPS (Receiver + ULF Antenna Connector)"
- note removed: "GPS (Receiver + SMA Antenna Connector)"
- moved on the sheet: R45

Commit message: MàJ 07/07/2025
Parts:
- R2: value 10R -> 10kR; footprint Resistor_10R_ERA-2AKD100X:RES_ERA2AKD100X -> Resistor_10kR_CRGP0402F10K:RESC1105X40N
Changed lines of the file:
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@@
 			)
 		)
-		(property "Datasheet" "GRM155C71H104JE19D"
+		(property "Datasheet" "GRM155C71H104JE19J"
 			(at 128.27 104.14 0)
 			(effects
@@
 				(path "/3db65ff8-efa4-4a5b-9e49-72b4834469e4/6bc3fe57-fc64-4617-9eb9-8962e5b37a5d"
 					(reference "#PWR3")
-					(unit 1)
-				)
-			)
-		)
-	)
-	(symbol
-		(lib_id "Resistor:R")
-		(at 193.04 72.39 0)
-		(unit 1)
-		(exclude_from_sim no)
-		(in_bom yes)
-		(on_board yes)
-		(dnp no)
-		(fields_autoplaced yes)
-		(property "Reference" "R2"
-			(at 195.58 71.1199 0)
-			(effects
-				(font
-					(size 1.27 1.27)
-				)
-				(justify left)
-			)
-		)
-		(property "Value" "10R"
-			(at 195.58 73.6599 0)
-			(effects
-				(font
-					(size 1.27 1.27)
-				)
-				(justify left)
-			)
-		)
-		(property "Footprint" "Resistor_10R_ERA-2AKD100X:RES_ERA2AKD100X"
-			(at 191.262 72.39 90)
-			(effects
-				(font
-					(size 1.27 1.27)
-				)
-				(hide yes)
-			)
-		)
-		(property "Datasheet" "ERA-2AKD100X"
-			(at 193.04 72.39 0)
-			(effects
-				(font
-					(size 1.27 1.27)
-				)
-				(hide yes)
-			)
-		)
-		(property "Description" "Resistor ERA-2AKD100X"
-			(at 193.04 72.39 0)
-			(effects
-				(font
-					(size 1.27 1.27)
-				)
-				(hide yes)
-			)
-		)
-		(pin "2"
-		)
-		(pin "1"
-		)
-		(instances
-			(project ""
-				(path "/3db65ff8-efa4-4a5b-9e49-72b4834469e4/6bc3fe57-fc64-4617-9eb9-8962e5b37a5d"
-					(reference "R2")
 					(unit 1)
 				)
@@
 					(unit 1)
 				)
+			)
+		)
+	)
+	(symbol
+		(lib_id "Resistor:R")
+		(at 193.04 72.39 0)
+		(unit 1)
+		(exclude_from_sim no)
+		(in_bom yes)
+		(on_board yes)
+		(dnp no)
+		(fields_autoplaced yes)
+		(property "Reference" "R2"
+			(at 195.58 71.1199 0)
+			(effects
+				(font
+					(size 1.27 1.27)
+				)
+				(justify left)
+			)
+		)
+		(property "Value" "10kR"
+			(at 195.58 73.6599 0)
+			(effects
+				(font
+					(size 1.27 1.27)
+				)
+				(justify left)
+			)
+		)
+		(property "Footprint" "Resistor_10kR_CRGP0402F10K:RESC1105X40N"
+			(at 191.262 72.39 90)
+			(effects
+				(font
+					(size 1.27 1.27)
+				)
+				(hide yes)
+			)
+		)
+		(property "Datasheet" "CRGP0402F10K"
+			(at 193.04 72.39 0)
+			(effects
+				(font
+					(size 1.27 1.27)
+				)
+				(hide yes)
+			)
+		)
+		(property "Description" "Resistor CRGP0402F10K"
+			(at 193.04 72.39 0)
+			(effects
+				(font
+					(size 1.27 1.27)
+				)
+				(hide yes)
+			)
+		)
+		(pin "2"
+		)
+		(pin "1"
+		)
+		(instances
+			(project "Card_CRAN_SEGULA"
+				(path "/3db65ff8-efa4-4a5b-9e49-72b4834469e4/6bc3fe57-fc64-4617-9eb9-8962e5b37a5d"
+					(reference "R2")
+					(unit 1)
+				)
